File: Hardware/Mood-Light-Perhaps.brd (EAGLE design)
At the start: 160 x 100 mm, 8 parts, among them U1 ATMEGA328P_TQFP, Y1 8MHz

Commit message: Progress made
Parts:
- added LED1: (no value), LinnesLab-Displays:DOTMATRIX_BL-M12A881UR
- added R2, R3, R4, R5, R6, R7, R8, R9: (no value), LinnesLab-Passives:R0603
Connections:
- new net ACTION: U1.19
- new net LD1: R6.1, U1.2
- new net LD10: LED1.10, U1.16
- new net LD11: LED1.11, U1.15
- new net LD12: R5.1, U1.14
- new net LD13: LED1.13, U1.13
- new net LD14: R3.1, U1.12
- new net LD15: LED1.15, U1.11
- new net LD16: LED1.16, U1.10
- new net LD2: R8.1, U1.1
- new net LD3: LED1.3, U1.32
- new net LD4: LED1.4, U1.28
- new net LD5: R9.1, U1.27
- new net LD6: LED1.6, U1.26
- new net LD7: R7.1, U1.25
- new net LD8: R4.1, U1.24
- new net LD9: R2.1, U1.17
- new net LEFT: U1.23
- new net MODE: U1.9
- new net N$1: LED1.9, R2.2
- new net N$10: LED1.5, R9.2
- new net N$4: LED1.14, R3.2
- new net N$5: LED1.8, R4.2
- new net N$6: LED1.12, R5.2
- new net N$7: LED1.1, R6.2
- new net N$8: LED1.7, R7.2
- new net N$9: LED1.2, R8.2
- new net RIGHT: U1.22
- new net RXD: U1.30
- new net TXD: U1.31
Changed lines of the file:
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@@
 <attribute name="VALUE" x="-13.335" y="-23.495" size="0.7112" layer="27"/>
+</element>
+<element name="LED1" library="LinnesLab-Displays" package="DOTMATRIX_BL-M12A881UR" value="" x="-31.75" y="-5.08" smashed="yes">
+<attribute name="NAME" x="-47.75" y="11.92" size="1.27" layer="25"/>
+<attribute name="VALUE" x="-47.75" y="-23.08" size="1.27" layer="27"/>
+</element>
+<element name="R2" library="LinnesLab-Passives" package="R0603" package3d_urn="urn:adsk.eagle:package:15661944/2" value="" x="-49.53" y="-26.67" smashed="yes">
+<attribute name="NAME" x="-50.165" y="-26.035" size="0.7112" layer="25"/>
+<attribute name="VALUE" x="-50.165" y="-28.575" size="0.7112" layer="27"/>
+</element>
+<element name="R3" library="LinnesLab-Passives" package="R0603" package3d_urn="urn:adsk.eagle:package:15661944/2" value="" x="-49.53" y="-30.48" smashed="yes">
+<attribute name="NAME" x="-50.165" y="-29.845" size="0.7112" layer="25"/>
+<attribute name="VALUE" x="-50.165" y="-32.385" size="0.7112" layer="27"/>
+</element>
+<element name="R4" library="LinnesLab-Passives" package="R0603" package3d_urn="urn:adsk.eagle:package:15661944/2" value="" x="-49.53" y="-34.29" smashed="yes">
+<attribute name="NAME" x="-50.165" y="-33.655" size="0.7112" layer="25"/>
+<attribute name="VALUE" x="-50.165" y="-36.195" size="0.7112" layer="27"/>
+</element>
+<element name="R5" library="LinnesLab-Passives" package="R0603" package3d_urn="urn:adsk.eagle:package:15661944/2" value="" x="-49.53" y="-38.1" smashed="yes">
+<attribute name="NAME" x="-50.165" y="-37.465" size="0.7112" layer="25"/>
+<attribute name="VALUE" x="-50.165" y="-40.005" size="0.7112" layer="27"/>
+</element>
+<element name="R6" library="LinnesLab-Passives" package="R0603" package3d_urn="urn:adsk.eagle:package:15661944/2" value="" x="-49.53" y="-41.91" smashed="yes">
+<attribute name="NAME" x="-50.165" y="-41.275" size="0.7112" layer="25"/>
+<attribute name="VALUE" x="-50.165" y="-43.815" size="0.7112" layer="27"/>
+</element>
+<element name="R7" library="LinnesLab-Passives" package="R0603" package3d_urn="urn:adsk.eagle:package:15661944/2" value="" x="-49.53" y="-45.72" smashed="yes">
+<attribute name="NAME" x="-50.165" y="-45.085" size="0.7112" layer="25"/>
+<attribute name="VALUE" x="-50.165" y="-47.625" size="0.7112" layer="27"/>
+</element>
+<element name="R8" library="LinnesLab-Passives" package="R0603" package3d_urn="urn:adsk.eagle:package:15661944/2" value="" x="-49.53" y="-49.53" smashed="yes">
+<attribute name="NAME" x="-50.165" y="-48.895" size="0.7112" layer="25"/>
+<attribute name="VALUE" x="-50.165" y="-51.435" size="0.7112" layer="27"/>
+</element>
+<element name="R9" library="LinnesLab-Passives" package="R0603" package3d_urn="urn:adsk.eagle:package:15661944/2" value="" x="-49.53" y="-53.34" smashed="yes">
+<attribute name="NAME" x="-50.165" y="-52.705" size="0.7112" layer="25"/>
+<attribute name="VALUE" x="-50.165" y="-55.245" size="0.7112" layer="27"/>
 </element>
 </elements>
@@
 <contactref element="C3" pad="1"/>
 </signal>
+<signal name="LEFT">
+<contactref element="U1" pad="23"/>
+</signal>
+<signal name="LD8">
+<contactref element="U1" pad="24"/>
+<contactref element="R4" pad="1"/>
+<wire x1="-0.7874" y1="10.42" x2="-50.38" y2="-34.29" width="0" layer="19" extent="1-1"/>
+</signal>
+<signal name="LD7">
+<contactref element="U1" pad="25"/>
+<contactref element="R7" pad="1"/>
+<wire x1="-2.28" y1="11.9126" x2="-50.38" y2="-45.72" width="0" layer="19" extent="1-1"/>
+</signal>
+<signal name="LD6">
+<contactref element="U1" pad="26"/>
+<contactref element="LED1" pad="6"/>
+<wire x1="-3.08" y1="11.9126" x2="-27.94" y2="-17.08" width="0" layer="19" extent="1-1"/>
+</signal>
+<signal name="LD5">
+<contactref element="U1" pad="27"/>
+<contactref element="R9" pad="1"/>
+<wire x1="-3.88" y1="11.9126" x2="-50.38" y2="-53.34" width="0" layer="19" extent="1-1"/>
+</signal>
+<signal name="LD4">
+<contactref element="U1" pad="28"/>
+<contactref element="LED1" pad="4"/>
+<wire x1="-4.68" y1="11.9126" x2="-33.02" y2="-17.08" width="0" layer="19" extent="1-1"/>
+</signal>
+<signal name="ACTION">
+<contactref element="U1" pad="19"/>
+</signal>
+<signal name="RIGHT">
+<contactref element="U1" pad="22"/>
+</signal>
+<signal name="RXD">
+<contactref element="U1" pad="30"/>
+</signal>
+<signal name="TXD">
+<contactref element="U1" pad="31"/>
+</signal>
+<signal name="LD3">
+<contactref element="U1" pad="32"/>
+<contactref element="LED1" pad="3"/>
+<wire x1="-7.88" y1="11.9126" x2="-35.56" y2="-17.08" width="0" layer="19" extent="1-1"/>
+</signal>
+<signal name="LD2">
+<contactref element="U1" pad="1"/>
+<contactref element="R8" pad="1"/>
+<wire x1="-9.3726" y1="10.42" x2="-50.38" y2="-49.53" width="0" layer="19" extent="1-1"/>
+</signal>
+<signal name="LD1">
+<contactref element="U1" pad="2"/>
+<contactref element="R6" pad="1"/>
+<wire x1="-9.3726" y1="9.62" x2="-50.38" y2="-41.91" width="0" layer="19" extent="1-1"/>
+</signal>
+<signal name="MODE">
+<contactref element="U1" pad="9"/>
+</signal>
+<signal name="LD16">
+<contactref element="U1" pad="10"/>
+<contactref element="LED1" pad="16"/>
+<wire x1="-7.08" y1="3.3274" x2="-40.64" y2="6.92" width="0" layer="19" extent="1-1"/>
+</signal>
+<signal name="LD15">
+<contactref element="U1" pad="11"/>
+<contactref element="LED1" pad="15"/>
+<wire x1="-6.28" y1="3.3274" x2="-38.1" y2="6.92" width="0" layer="19" extent="1-1"/>
+</signal>
+<signal name="LD14">
+<contactref element="U1" pad="12"/>
+<contactref element="R3" pad="1"/>
+<wire x1="-5.48" y1="3.3274" x2="-50.38" y2="-30.48" width="0" layer="19" extent="1-1"/>
+</signal>
+<signal name="LD13">
+<contactref element="U1" pad="13"/>
+<contactref element="LED1" pad="13"/>
+<wire x1="-4.68" y1="3.3274" x2="-33.02" y2="6.92" width="0" layer="19" extent="1-1"/>
+</signal>
+<signal name="LD12">
+<contactref element="U1" pad="14"/>
+<contactref element="R5" pad="1"/>
+<wire x1="-3.88" y1="3.3274" x2="-50.38" y2="-38.1" width="0" layer="19" extent="1-1"/>
+</signal>
+<signal name="LD11">
+<contactref element="U1" pad="15"/>
+<contactref element="LED1" pad="11"/>
+<wire x1="-3.08" y1="3.3274" x2="-27.94" y2="6.92" width="0" layer="19" extent="1-1"/>
+</signal>
+<signal name="LD10">
+<contactref element="U1" pad="16"/>
+<contactref element="LED1" pad="10"/>
+<wire x1="-2.28" y1="3.3274" x2="-25.4" y2="6.92" width="0" layer="19" extent="1-1"/>
+</signal>
+<signal name="LD9">
+<contactref element="U1" pad="17"/>
+<contactref element="R2" pad="1"/>
+<wire x1="-0.7874" y1="4.82" x2="-50.38" y2="-26.67" width="0" layer="19" extent="1-1"/>
+</signal>
+<signal name="N$1">
+<contactref element="LED1" pad="9"/>
+<contactref element="R2" pad="2"/>
+<wire x1="-22.86" y1="6.92" x2="-48.68" y2="-26.67" width="0" layer="19" extent="1-1"/>
+</signal>
+<signal name="N$4">
+<contactref element="LED1" pad="14"/>
+<contactref element="R3" pad="2"/>
+<wire x1="-35.56" y1="6.92" x2="-48.68" y2="-30.48" width="0" layer="19" extent="1-1"/>
+</signal>
+<signal name="N$5">
+<contactref element="LED1" pad="8"/>
+<contactref element="R4" pad="2"/>
+<wire x1="-22.86" y1="-17.08" x2="-48.68" y2="-34.29" width="0" layer="19" extent="1-1"/>
+</signal>
+<signal name="N$6">
+<contactref element="LED1" pad="12"/>
+<contactref element="R5" pad="2"/>
+<wire x1="-30.48" y1="6.92" x2="-48.68" y2="-38.1" width="0" layer="19" extent="1-1"/>
+</signal>
+<signal name="N$7">
+<contactref element="LED1" pad="1"/>
+<contactref element="R6" pad="2"/>
+<wire x1="-40.64" y1="-17.08" x2="-48.68" y2="-41.91" width="0" layer="19" extent="1-1"/>
+</signal>
+<signal name="N$8">
+<contactref element="LED1" pad="7"/>
+<contactref element="R7" pad="2"/>
+<wire x1="-25.4" y1="-17.08" x2="-48.68" y2="-45.72" width="0" layer="19" extent="1-1"/>
+</signal>
+<signal name="N$9">
+<contactref element="LED1" pad="2"/>
+<contactref element="R8" pad="2"/>
+<wire x1="-38.1" y1="-17.08" x2="-48.68" y2="-49.53" width="0" layer="19" extent="1-1"/>
+</signal>
+<signal name="N$10">
+<contactref element="LED1" pad="5"/>
+<contactref element="R9" pad="2"/>
+<wire x1="-30.48" y1="-17.08" x2="-48.68" y2="-53.34" width="0" layer="19" extent="1-1"/>
+</signal>
 </signals>

Commit message: Finished schematic
Parts:
- added C6, C7: 1u, LinnesLab-Passives:C0603
- added C8, C9: 4.7u, LinnesLab-Passives:C0603
- added D1, D2: (no value), LinnesLab-DiscreteSemi:USC
- added J1: FTDI_DEVICE, LinnesLab-Connectors:FTDI_DEVICE
- added J2: AVR_SPI_PROG_3X2NS, LinnesLab-Connectors:2X3-NS
- added LED2: (no value), LinnesLab-LED:LED_5MM
- added LIPO1: (no value), LinnesLab-Connectors:JST-2-SMD
- added R10, R11, R12: 10k, LinnesLab-Passives:R0603
- added R13: 100k, LinnesLab-Passives:R0603
- added R14: (no value), LinnesLab-Passives:R0603
- added SW1, SW2, SW3: (no value), LinnesLab-Switches:SPST.KT11P4SM34LFS
- added SW4, SW5: SWITCH.JS202011JXQNUPWARDS, LinnesLab-Switches:SWITCH.00
- added U2: MCP73831.SOT23-5, LinnesLab-Power:SOT23-5
- added U3: MIC550X, LinnesLab-Power:SOT23-5
- added USB1: USB.MICRO-BIGGERPADS, LinnesLab-Connectors:USB-MICRO-01.BIGGERPADS
- R2, R3, R4, R5, R6, R7, R8, R9: value (none) -> 205
Connections:
- new net CHRG.STAT: LED2.A, R13.1
- new net N$11: R12.1
- new net N$12: R14.2, U2.5
- new net N$13: D1.+, SW5.1
- new net N$16: LED2.K, U2.1
- new net VIN: C6.1, C8.1, D1.-, D2.-, R13.2, U2.4, U3.1, U3.3
- new net VLIPO: C9.1, LIPO1.2, SW5.2, U2.3
- new net V_USB: D2.+, USB1.1
- net 3.3V: now also C7.1, J1.VCC, J2.2, SW1.1, SW1.2, SW2.1, SW2.2, SW3.1, SW3.2, SW4.1, U3.5
- net ACTION: now also R12.2, SW3.3, SW3.4
- net DTR: now also J1.DTR
- net GND: now also C6.2, C7.2, C8.2, C9.2, J1.CTS, J1.GND, J2.6, LIPO1.1, R10.1, R11.1, R14.1, SW4.3, U2.2, U3.2, USB1.5, USB1.S1, USB1.S2, USB1.S3, USB1.S4, USB1.S5, USB1.S6
- net LD10: now also J2.1
- net LD11: now also J2.4
- net LD9: now also J2.3
- net LEFT: now also R10.2, SW1.3, SW1.4
- net MODE: now also SW4.2
- net RESET: now also J2.5
- net RIGHT: now also R11.2, SW2.3, SW2.4
- net RXD: now also J1.RXI
- net TXD: now also J1.TXO

Commit message: Board progress 1
Parts:
- moved C7 257.5 mm to (105.4, 38.1)
- moved C6 256.5 mm to (105.4, 40.6)
- moved R13 256.5 mm to (105.4, 25.4)
- moved LIPO1 255.7 mm to (111.8, 50.8)
- moved C8 255.7 mm to (104.1, 29.2)
- moved C9 255.7 mm to (97.8, 15.2)
- moved D2 255.7 mm to (104.1, 33.0)
- moved SW5 255.7 mm to (121.9, 50.8)
- moved D1 255.7 mm to (104.1, 45.7)
- moved LED2 255.7 mm to (99.1, 27.9)
- moved R14 255.7 mm to (97.8, 20.3)
- moved U2 255.7 mm to (119.4, 62.2)
- moved U3 255.7 mm to (119.4, 55.9)
- moved USB1 255.7 mm to (121.9, 68.6)
- moved J1 218.8 mm to (137.2, 66.0)
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
Commit message: Board progress 2
Parts:
- moved SW4 63.1 mm to (73.7, 33.0)
- moved U2 40.5 mm to (97.8, 27.9), turned to 270 degrees
- moved C3 16.1 mm to (76.2, 52.1), turned to 90 degrees
- moved R13 15.2 mm to (90.2, 25.4)
- moved C8 10.5 mm to (101.6, 19.1)
- moved R14 9.67 mm to (101.6, 29.2), turned to 180 degrees
- moved LED2 9.25 mm to (90.2, 30.5)
- moved C9 8.98 mm to (96.5, 24.1), turned to 270 degrees
- moved R1 6.35 mm to (76.2, 55.9), turned to 90 degrees

Commit message: Changed LED
Parts:
- removed LED2: (no value), LinnesLab-LED:LED_5MM
- added LED3: (no value), LinnesLab-LED:LED-0805
Connections:
- net CHRG.STAT: now also LED3.A; no longer LED2.A
- net N$16: now also LED3.C; no longer LED2.K
Changed lines of the file:
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@@
 <attribute name="VALUE" x="89.535" y="23.495" size="0.7112" layer="27"/>
-</element>
-<element name="LED2" library="LinnesLab-LED" package="LED_5MM" value="" x="90.17" y="30.48" smashed="yes">
-<attribute name="NAME" x="90.17" y="33.8709" size="0.7112" layer="25" ratio="20" align="bottom-center"/>
-<attribute name="VALUE" x="90.1954" y="27.0891" size="0.7112" layer="27" ratio="20" align="top-center"/>
 </element>
 <element name="R14" library="LinnesLab-Passives" package="R0603" package3d_urn="urn:adsk.eagle:package:15661944/2" value="" x="101.6" y="29.21" smashed="yes" rot="R180">
@@
 <attribute name="NAME" x="97.155" y="24.765" size="0.7112" layer="25" rot="R270"/>
 <attribute name="VALUE" x="94.615" y="24.765" size="0.7112" layer="27" rot="R270"/>
+</element>
+<element name="LED3" library="LinnesLab-LED" package="LED-0805" value="" x="92.71" y="31.75" smashed="yes">
+<attribute name="NAME" x="91.44" y="30.48" size="1.27" layer="25" rot="R90"/>
+<attribute name="VALUE" x="95.25" y="30.48" size="1.27" layer="27" rot="R90"/>
 </element>
 </elements>
@@
 <signal name="CHRG.STAT">
 <contactref element="R13" pad="1"/>
-<contactref element="LED2" pad="A"/>
-<wire x1="89.32" y1="25.4" x2="88.9" y2="30.48" width="0" layer="19" extent="1-1"/>
+<contactref element="LED3" pad="A"/>
+<wire x1="92.71" y1="30.7" x2="89.32" y2="25.4" width="0" layer="19" extent="1-1"/>
 </signal>
 <signal name="N$16">
-<contactref element="LED2" pad="K"/>
 <contactref element="U2" pad="1"/>
-<wire x1="96.4899" y1="28.89" x2="91.44" y2="30.48" width="0" layer="19" extent="1-1"/>
+<contactref element="LED3" pad="C"/>
+<wire x1="92.71" y1="32.8" x2="96.4899" y2="28.89" width="0" layer="19" extent="1-1"/>
 </signal>
 </signals>

Commit message: Progress 3
Parts:
- R14: value (none) -> 2k
- moved J2 111.0 mm to (22.5, 53.3)
- moved SW2 102.7 mm to (31.3, 25.0), turned to 270 degrees
- moved SW3 102.7 mm to (31.2, 13.4), turned to 270 degrees
- moved SW1 102.6 mm to (31.3, 38.9), turned to 270 degrees
- moved R10 100.8 mm to (28.8, 46.6)
- moved R12 100.0 mm to (30.5, 5.31), turned to 180 degrees
- moved R11 99.5 mm to (30.0, 32.0), turned to 180 degrees
- moved J1 95.6 mm to (50.2, 26.3), turned to 180 degrees
- moved USB1 65.5 mm to (110.9, 4.01)
- moved LIPO1 47.5 mm to (122.7, 4.57), turned to 180 degrees
- moved R1 35.6 mm to (50.1, 31.6), turned to 0 degrees
- moved C3 34.5 mm to (50.1, 29.4), turned to 180 degrees
- moved C7 33.7 mm to (78.7, 17.4)
- moved SW5 33.0 mm to (121.5, 17.8)
- moved LED1 29.5 mm to (51.0, 72.5)
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Routing:
- net LD16: track 0.00 -> 17.1 mm
- net LD15: track 0.00 -> 16.4 mm
- net LD10: track 0.00 -> 15.5 mm
- net LD13: track 0.00 -> 14.9 mm
- net LD11: track 0.00 -> 14.8 mm
- net LD2: track 0.00 -> 9.69 mm
- net N$5: track 0.00 -> 8.80 mm
- net N$9: track 0.00 -> 8.58 mm
- net N$8: track 0.00 -> 8.34 mm
- net N$10: track 0.00 -> 8.32 mm
- net N$7: track 0.00 -> 8.31 mm
- net LD14: track 0.00 -> 7.76 mm
- net LD12: track 0.00 -> 6.32 mm
- net N$6: track 0.00 -> 6.20 mm
- net N$4: track 0.00 -> 6.20 mm
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
Commit message: Progress 4
Parts:
- moved C4 54.2 mm to (131.8, 4.52)
- moved C5 54.2 mm to (131.8, 2.79)
- moved C7 54.2 mm to (131.8, 6.25)
- moved R12 34.3 mm to (23.7, 38.9), turned to 90 degrees
- moved SW3 32.1 mm to (18.2, 42.7), turned to 90 degrees
- moved C9 25.9 mm to (122.5, 12.2), turned to 0 degrees
- moved SW1 23.7 mm to (18.3, 19.1), turned to 90 degrees
- moved R10 23.6 mm to (23.6, 23.5), turned to 90 degrees
- moved U3 22.8 mm to (112.2, 9.12)
- moved C6 17.1 mm to (116.2, 11.4)
- moved D1 17.1 mm to (116.2, 13.5)
- moved LED3 16.6 mm to (95.8, 3.12)
- moved SW2 14.2 mm to (18.3, 30.7), turned to 90 degrees
- moved R14 13.6 mm to (103.5, 3.43), turned to 90 degrees
- moved D2 13.2 mm to (108.1, 8.18)
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Routing:
- net RESET: track 0.00 -> 100.0 mm
- net LD3: track 0.00 -> 80.5 mm
- net VLIPO: track 0.00 -> 79.1 mm
- net LD4: track 0.00 -> 64.4 mm, vias 0 -> 2
- net LD8: track 0.00 -> 61.7 mm, vias 0 -> 2
- net LD7: track 0.00 -> 60.3 mm, vias 0 -> 2
- net LD5: track 0.00 -> 60.1 mm, vias 0 -> 2
- net LD1: track 0.85 -> 57.1 mm, vias 0 -> 1
- net LD6: track 0.00 -> 51.9 mm, vias 0 -> 1
- net LD2: track 9.69 -> 56.4 mm, vias 0 -> 2
- net LEFT: track 0.00 -> 41.3 mm
- net RIGHT: track 0.00 -> 36.9 mm
- net ACTION: track 0.00 -> 36.4 mm
- net VIN: track 0.00 -> 35.4 mm
- net LD9: track 0.00 -> 29.8 mm
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
Commit message: Progress 6? need to fix errors
Parts:
- moved LIPO1 47.6 mm to (75.1, 3.15)
- moved C6 47.6 mm to (68.6, 11.5)
- moved D1 47.6 mm to (68.6, 13.6)
- moved R13 47.6 mm to (43.0, 2.95)
- moved U3 47.6 mm to (64.6, 9.14)
- moved LED3 47.6 mm to (48.2, 3.15)
- moved R14 47.6 mm to (55.9, 3.45)
- moved C4 47.6 mm to (84.2, 4.55)
- moved C5 47.6 mm to (84.2, 2.82)
- moved C7 47.6 mm to (84.2, 6.27)
- moved C8 47.6 mm to (45.2, 2.97)
- moved C9 47.6 mm to (74.9, 12.2)
- moved D2 47.6 mm to (60.5, 8.20)
- moved SW5 47.6 mm to (73.9, 17.9)
- moved U2 47.6 mm to (52.2, 3.07)
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Routing:
- net 3.3V: track 0.00 -> 161.5 mm, vias 0 -> 4
- net GND: track 0.00 -> 85.7 mm, vias 0 -> 12
- net RXD: track 11.6 -> 48.0 mm, vias 0 -> 2
- net VLIPO: track 79.1 -> 44.8 mm
- net TXD: track 12.0 -> 43.1 mm, vias 0 -> 2
- net DTR: track 10.9 -> 32.9 mm
- net LD4: track 64.4 -> 52.4 mm, vias 2 -> 1
- net VIN: track 35.4 -> 37.4 mm
- added copper zone on layer 1, net 3.3V
- added copper zone on layer 16, net GND
Other:
- board size 160 x 100 mm -> 100 x 100 mm
