File: Hardware/Mood-Light-Perhaps.brd (EAGLE design)
At the start: 100 x 100 mm, 40 parts, among them J1 FTDI_DEVICE, J2 AVR_SPI_PROG_3X2NS, SW4 SWITCH.JS202011JXQNUPWARDS, SW5 SWITCH.JS202011JXQNUPWARDS, U1 ATMEGA328P_TQFP, U2 MCP73831.SOT23-5, U3 MIC550X, Y1 8MHz

Commit message: Completed PCB
Routing:
- net 3.3V: track 161.5 -> 80.4 mm
- net GND: track 85.7 -> 92.2 mm, vias 12 -> 13
- net LD2: track 56.4 -> 60.2 mm
- net LD1: vias 1 -> 0

Commit message: edited board and added CAM outputs
Parts:
- moved USB1 1.22 mm to (63.3, 2.82)
- moved J1 0.38 mm to (32.4, 1.98)
- moved LIPO1 0.15 mm to (75.1, 3.30)
Connections:
- removed net N$11: R12.1
- net GND: now also R12.1
Routing:
- net RESET: track 100.0 -> 42.8 mm, vias 0 -> 1
- net 3.3V: track 80.4 -> 25.5 mm, vias 4 -> 3
- net GND: track 92.2 -> 76.4 mm, vias 13 -> 15
- net VLIPO: track 44.8 -> 39.5 mm, vias 0 -> 2
- net VIN: track 37.4 -> 40.2 mm
- net V_USB: track 2.81 -> 4.03 mm
- net N$13: track 3.35 -> 3.99 mm

Commit message: updated GERBERs for FTDI silkscreen
Parts:
- moved J1 0.64 mm to (32.4, 2.62)
Routing:
- net RXD: track 47.6 -> 47.0 mm
- net DTR: track 32.5 -> 31.9 mm
- net TXD: track 42.7 -> 42.1 mm
Changed lines of the file:
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@@
 <attribute name="VALUE" x="48.3616" y="90.9066" size="0.7112" layer="27"/>
 </element>
-<element name="J1" library="LinnesLab-Connectors" package="FTDI_DEVICE" value="FTDI_DEVICE" x="32.385" y="1.9812" smashed="yes" rot="R180"/>
+<element name="J1" library="LinnesLab-Connectors" package="FTDI_DEVICE" value="FTDI_DEVICE" x="32.3596" y="2.6162" smashed="yes" rot="R180"/>
 <element name="J2" library="LinnesLab-Connectors" package="2X3-NS" package3d_urn="urn:adsk.eagle:package:18167648/2" value="AVR_SPI_PROG_3X2NS" x="22.5298" y="53.2638" smashed="yes">
 <attribute name="NAME" x="21.5138" y="56.2356" size="0.7112" layer="25" ratio="20"/>
@@
 <contactref element="C3" pad="1"/>
 <contactref element="J1" pad="DTR"/>
-<wire x1="50.9642" y1="29.4386" x2="38.735" y2="17.2094" width="0.1524" layer="1"/>
-<wire x1="38.735" y1="17.2094" x2="38.735" y2="1.9812" width="0.1524" layer="1"/>
+<wire x1="50.9642" y1="29.4386" x2="38.7096" y2="17.184" width="0.1524" layer="1"/>
+<wire x1="38.7096" y1="17.184" x2="38.7096" y2="2.6162" width="0.1524" layer="1"/>
 </signal>
 <signal name="LEFT">
@@
 <contactref element="U1" pad="30"/>
 <contactref element="J1" pad="RXI"/>
-<wire x1="33.655" y1="1.9812" x2="33.655" y2="4.4958" width="0.1524" layer="1"/>
-<wire x1="33.655" y1="4.4958" x2="33.782" y2="4.6228" width="0.1524" layer="1"/>
+<wire x1="33.6296" y1="2.6162" x2="33.6296" y2="4.4704" width="0.1524" layer="1"/>
+<wire x1="33.6296" y1="4.4704" x2="33.782" y2="4.6228" width="0.1524" layer="1"/>
 <via x="33.782" y="4.6228" extent="1-16" drill="0.35"/>
 <via x="51.9176" y="36.2712" extent="1-16" drill="0.35"/>
@@
 <contactref element="U1" pad="31"/>
 <contactref element="J1" pad="TXO"/>
-<wire x1="36.195" y1="1.9812" x2="36.195" y2="5.0292" width="0.1524" layer="1"/>
-<wire x1="36.195" y1="5.0292" x2="36.3982" y2="5.2324" width="0.1524" layer="1"/>
+<wire x1="36.1696" y1="2.6162" x2="36.1696" y2="5.0038" width="0.1524" layer="1"/>
+<wire x1="36.1696" y1="5.0038" x2="36.3982" y2="5.2324" width="0.1524" layer="1"/>
 <via x="36.3982" y="5.2324" extent="1-16" drill="0.35"/>
 <wire x1="36.3982" y1="5.2324" x2="36.3982" y2="19.6342" width="0.1524" layer="16"/>
