File: Hardware/Mood-Light-Perhaps.sch (EAGLE design)
At the start: 8 parts, among them U1 ATMEGA328P_TQFP, Y1 8MHz

Commit message: Progress made
Parts:
- added LED1: (no value), LinnesLab-Displays:DOTMATRIX_8X8_ROWCATHODEM12A881UR
- added R2, R3, R4, R5, R6, R7, R8, R9: (no value), LinnesLab-Passives:RESISTOR0603
Connections:
- new net ACTION: U1.ADC6
- new net LD1: R6.1, U1.D4/PD4(XCK/T0)
- new net LD10: LED1.A4, U1.D12/PB4(MISO)
- new net LD11: LED1.A6, U1.D11/PB3(MOSI/OC2)
- new net LD12: R5.1, U1.D10/PB2(SS/OC1B)
- new net LD13: LED1.A1, U1.D9/PB1(OC1A)
- new net LD14: R3.1, U1.D8/PB0(ICP)
- new net LD15: LED1.A7, U1.D7/PD7(AIN1)
- new net LD16: LED1.A8, U1.D6/PD6(AIN0)
- new net LD2: R8.1, U1.D3/PD3(INT1)
- new net LD3: LED1.A2, U1.D2/PD2(INT0)
- new net LD4: LED1.A3, U1.PC5(ADC5/SCL)
- new net LD5: R9.1, U1.PC4(ADC4/SDA)
- new net LD6: LED1.A5, U1.PC3(ADC3)
- new net LD7: R7.1, U1.PC2(ADC2)
- new net LD8: R4.1, U1.PC1(ADC1)
- new net LD9: R2.1, U1.D13/PB5(SCK)
- new net LEFT: U1.PC0(ADC0)
- new net MODE: U1.D5/PD5(T1)
- new net N$1: LED1.K1, R2.2
- new net N$10: LED1.K8, R9.2
- new net N$4: LED1.K2, R3.2
- new net N$5: LED1.K3, R4.2
- new net N$6: LED1.K4, R5.2
- new net N$7: LED1.K5, R6.2
- new net N$8: LED1.K6, R7.2
- new net N$9: LED1.K7, R8.2
- new net RIGHT: U1.ADC7
- new net RXD: U1.D0/PD0(RXD)
- new net TXD: U1.D1/PD1(TXD)

Commit message: Finished schematic
Parts:
- added C6, C7: 1u, LinnesLab-Passives:CAPACITOR0603
- added C8, C9: 4.7u, LinnesLab-Passives:CAPACITOR0603
- added D1, D2: (no value), LinnesLab-DiscreteSemi:SCHOTTKY-USC
- added J1: FTDI_DEVICE, LinnesLab-Connectors:FTDI_DEVICE
- added J2: AVR_SPI_PROG_3X2NS, LinnesLab-Connectors:AVR_SPI_PROG_3X2NS
- added LED2: (no value), LinnesLab-LED:LED5MM
- added LIPO1: (no value), LinnesLab-Connectors:JST_2MM_MALE
- added R10, R11, R12: 10k, LinnesLab-Passives:RESISTOR0603
- added R13: 100k, LinnesLab-Passives:RESISTOR0603
- added R14: (no value), LinnesLab-Passives:RESISTOR0603
- added SW1, SW2, SW3: (no value), LinnesLab-Switches:SPST.KT11P4SM34LFS
- added SW4, SW5: SWITCH.JS202011JXQNUPWARDS, LinnesLab-Switches:SWITCH.JS202011JXQNUPWARDS
- added U2: MCP73831.SOT23-5, LinnesLab-Power:MCP73831.SOT23-5
- added U3: MIC550X, LinnesLab-Power:MIC550X
- added USB1: USB.MICRO-BIGGERPADS, LinnesLab-Connectors:USB.MICRO-BIGGERPADS
- R2, R3, R4, R5, R6, R7, R8, R9: value (none) -> 205
Connections:
- new net CHRG.STAT: LED2.A, R13.1
- new net N$11: R12.1
- new net N$12: R14.2, U2.PROG
- new net N$13: D1.A, SW5.1
- new net N$16: LED2.C, U2.STAT
- new net VIN: C6.1, C8.1, D1.C, D2.C, R13.2, U2.VIN, U3.EN, U3.IN
- new net VLIPO: C9.1, LIPO1.+, SW5.2, U2.VBAT
- new net V_USB: D2.A, USB1.V+
- net 3.3V: now also C7.1, J1.VCC, J2.2, SW1.A, SW2.A, SW3.A, SW4.1, U3.OUT
- net ACTION: now also R12.2, SW3.B
- net DTR: now also J1.DTR
- net GND: now also C6.2, C7.2, C8.2, C9.2, J1.CTS, J1.GND, J2.6, LIPO1.-, R10.1, R11.1, R14.1, SW4.3, U2.VSS, U3.GND, USB1.GND, USB1.SHIELD
- net LD10: now also J2.1
- net LD11: now also J2.4
- net LD9: now also J2.3
- net LEFT: now also R10.2, SW1.B
- net MODE: now also SW4.2
- net RESET: now also J2.5
- net RIGHT: now also R11.2, SW2.B
- net RXD: now also J1.TXO
- net TXD: now also J1.RXI

Commit message: Changed LED
Parts:
- removed LED2: (no value), LinnesLab-LED:LED5MM
- added LED3: (no value), LinnesLab-LED:LED0805
Connections:
- net CHRG.STAT: now also LED3.A; no longer LED2.A
- net N$16: now also LED3.C; no longer LED2.C
Changed lines of the file:
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@@
 <part name="C8" library="LinnesLab-Passives" deviceset="CAPACITOR" device="0603" package3d_urn="urn:adsk.eagle:package:15661989/2" value="4.7u"/>
 <part name="R13" library="LinnesLab-Passives" deviceset="RESISTOR" device="0603" package3d_urn="urn:adsk.eagle:package:15661944/2" value="100k"/>
-<part name="LED2" library="LinnesLab-LED" deviceset="LED" device="5MM"/>
 <part name="R14" library="LinnesLab-Passives" deviceset="RESISTOR" device="0603" package3d_urn="urn:adsk.eagle:package:15661944/2"/>
 <part name="C9" library="LinnesLab-Passives" deviceset="CAPACITOR" device="0603" package3d_urn="urn:adsk.eagle:package:15661989/2" value="4.7u"/>
@@
 <part name="GND18" library="LinnesLab-Symbols" deviceset="GND" device=""/>
 <part name="SUPPLY14" library="LinnesLab-Symbols" deviceset="VLIPO" device=""/>
+<part name="LED3" library="LinnesLab-LED" deviceset="LED" device="0805"/>
 </parts>
 <sheets>
@@
 <attribute name="VALUE" x="69.342" y="-95.25" size="1.778" layer="96" rot="R90"/>
 </instance>
-<instance part="LED2" gate="G$1" x="76.2" y="-93.98" smashed="yes" rot="R180">
-<attribute name="NAME" x="79.629" y="-89.408" size="1.778" layer="95" font="vector" rot="R270"/>
-<attribute name="VALUE" x="74.295" y="-89.408" size="1.778" layer="96" font="vector" rot="R270" align="top-left"/>
-</instance>
 <instance part="R14" gate="G$1" x="111.76" y="-86.36" smashed="yes" rot="R90">
 <attribute name="NAME" x="110.2614" y="-90.17" size="1.778" layer="95" rot="R90"/>
@@
 <instance part="SUPPLY14" gate="G$1" x="119.38" y="-76.2" smashed="yes">
 <attribute name="VALUE" x="119.38" y="-73.406" size="1.778" layer="96" align="bottom-center"/>
+</instance>
+<instance part="LED3" gate="G$1" x="76.2" y="-91.44" smashed="yes" rot="R180">
+<attribute name="NAME" x="79.629" y="-86.868" size="1.778" layer="95" font="vector" rot="R270"/>
+<attribute name="VALUE" x="74.295" y="-86.868" size="1.778" layer="96" font="vector" rot="R270" align="top-left"/>
 </instance>
 </instances>
@@
 <wire x1="66.04" y1="-96.52" x2="66.04" y2="-99.06" width="0.1524" layer="91"/>
 <wire x1="66.04" y1="-99.06" x2="76.2" y2="-99.06" width="0.1524" layer="91"/>
-<pinref part="LED2" gate="G$1" pin="A"/>
-<wire x1="76.2" y1="-99.06" x2="76.2" y2="-96.52" width="0.1524" layer="91"/>
 <label x="81.28" y="-99.06" size="1.778" layer="95"/>
+<pinref part="LED3" gate="G$1" pin="A"/>
+<wire x1="76.2" y1="-99.06" x2="76.2" y2="-93.98" width="0.1524" layer="91"/>
 </segment>
 </net>
 <net name="N$16" class="0">
 <segment>
-<pinref part="LED2" gate="G$1" pin="C"/>
-<wire x1="76.2" y1="-88.9" x2="76.2" y2="-83.82" width="0.1524" layer="91"/>
 <pinref part="U2" gate="G$1" pin="STAT"/>
 <wire x1="76.2" y1="-83.82" x2="81.28" y2="-83.82" width="0.1524" layer="91"/>
-</segment>
-</net>
+<pinref part="LED3" gate="G$1" pin="C"/>
+<wire x1="76.2" y1="-86.36" x2="76.2" y2="-83.82" width="0.1524" layer="91"/>
+</segment>
+</net>

Commit message: Progress 3
Parts:
- R14: value (none) -> 2k
Changed lines of the file:
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@@
 <part name="C8" library="LinnesLab-Passives" deviceset="CAPACITOR" device="0603" package3d_urn="urn:adsk.eagle:package:15661989/2" value="4.7u"/>
 <part name="R13" library="LinnesLab-Passives" deviceset="RESISTOR" device="0603" package3d_urn="urn:adsk.eagle:package:15661944/2" value="100k"/>
-<part name="R14" library="LinnesLab-Passives" deviceset="RESISTOR" device="0603" package3d_urn="urn:adsk.eagle:package:15661944/2"/>
+<part name="R14" library="LinnesLab-Passives" deviceset="RESISTOR" device="0603" package3d_urn="urn:adsk.eagle:package:15661944/2" value="2k"/>
 <part name="C9" library="LinnesLab-Passives" deviceset="CAPACITOR" device="0603" package3d_urn="urn:adsk.eagle:package:15661989/2" value="4.7u"/>
 <part name="GND15" library="LinnesLab-Symbols" deviceset="GND" device=""/>

Commit message: edited board and added CAM outputs
Connections:
- removed net N$11: R12.1
- net GND: now also R12.1
Changed lines of the file:
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@@
 <part name="SUPPLY14" library="LinnesLab-Symbols" deviceset="VLIPO" device=""/>
 <part name="LED3" library="LinnesLab-LED" deviceset="LED" device="0805"/>
+<part name="GND19" library="LinnesLab-Symbols" deviceset="GND" device=""/>
 </parts>
 <sheets>
@@
 <attribute name="NAME" x="79.629" y="-86.868" size="1.778" layer="95" font="vector" rot="R270"/>
 <attribute name="VALUE" x="74.295" y="-86.868" size="1.778" layer="96" font="vector" rot="R270" align="top-left"/>
+</instance>
+<instance part="GND19" gate="G$1" x="132.08" y="-58.42" smashed="yes">
+<attribute name="VALUE" x="132.08" y="-58.674" size="1.778" layer="96" align="top-center"/>
 </instance>
 </instances>
@@
 <wire x1="58.42" y1="-96.52" x2="58.42" y2="-91.44" width="0.1524" layer="91"/>
 </segment>
+<segment>
+<pinref part="R12" gate="G$1" pin="1"/>
+<wire x1="132.08" y1="-55.88" x2="132.08" y2="-50.8" width="0.1524" layer="91"/>
+<pinref part="GND19" gate="G$1" pin="GND"/>
+</segment>
 </net>
 <net name="N$2" class="0">
@@
 </segment>
 </net>
-<net name="N$11" class="0">
-<segment>
-<pinref part="R12" gate="G$1" pin="1"/>
-<wire x1="132.08" y1="-55.88" x2="132.08" y2="-50.8" width="0.1524" layer="91"/>
-</segment>
-</net>
